Commit message: Updated tooling position

File: snp_ur3/urdf/workcell.xacro (robot description, xacro)
@@ -87,5 +87,5 @@
   </link>
   <joint name="tool0_to_ee" type="fixed">
-    <origin xyz="0 0 -0.006" rpy="0 0 ${radians(-17)}"/>
+    <origin xyz="0 0 -0.006" rpy="0 0 ${radians(73)}"/>
     <parent link="tool0"/>
     <child link="ee"/>
@@ -94,5 +94,5 @@
   <link name="camera_color_optical_frame"/>
   <joint name="tool0_to_camera" type="fixed">
-    <parent link="tool0"/>
+    <parent link="ee"/>
     <child link="camera_color_optical_frame"/>
     <origin xyz="${camera_cal['camera_mount_to_camera_pos']['x']} ${camera_cal['camera_mount_to_camera_pos']['y']} ${camera_cal['camera_mount_to_camera_pos']['z']}"

Commit message: Updated calibration file

File: snp_ur3/urdf/workcell.xacro (robot description, xacro)
@@ -91,8 +91,8 @@
     <child link="ee"/>
   </joint>
-  <xacro:property name="camera_cal" value="${load_yaml('$(find snp_ur3)/config/camera_calibration.yaml')}" />
+  <xacro:property name="camera_cal" value="${load_yaml('$(find snp_ur3)/config/calibration.yaml')}" />
   <link name="camera_color_optical_frame"/>
   <joint name="tool0_to_camera" type="fixed">
-    <parent link="ee"/>
+    <parent link="tool0"/>
     <child link="camera_color_optical_frame"/>
     <origin xyz="${camera_cal['camera_mount_to_camera_pos']['x']} ${camera_cal['camera_mount_to_camera_pos']['y']} ${camera_cal['camera_mount_to_camera_pos']['z']}"

Commit message: Updated TCP location

File: snp_ur3/urdf/workcell.xacro (robot description, xacro)
@@ -111,5 +111,5 @@
     <parent link="ee"/>
     <child link="sand_tcp"/>
-    <origin xyz="0 0.05 0.025" rpy="${radians(-90)} 0 0"/>
+    <origin xyz="0 ${1.75 * 0.0254} 0.025" rpy="${radians(-90)} 0 0"/>
   </joint>
 </robot>

Commit message: Removed table top collision object

File: snp_ur3/urdf/workcell.xacro (robot description, xacro)
@@ -56,10 +56,4 @@
       </geometry>
     </collision>
-    <collision>
-      <origin xyz="0 0 0.726" rpy="0 0 0"/>
-      <geometry>
-        <box size="1.9 0.95 0.05"/>
-      </geometry>
-    </collision>
   </link>
   <joint name="floor_to_table" type="fixed">
